Commit message: Update src packages for HRVO navigation (lookahead 4m, fusion sync)

File: src/velodyne_simulator/velodyne_description/urdf/VLP-16.urdf.xacro (robot description, xacro)
@@ -2,5 +2,5 @@
 <robot xmlns:xacro="http://www.ros.org/wiki/xacro" name="VLP-16">
   <xacro:property name="M_PI" value="3.1415926535897931" />
-  <xacro:macro name="VLP-16" params="*origin parent:=upper_base_link name:=velodyne topic:=/velodyne_points hz:=20 lasers:=16 samples:=440 collision_range:=0.3 min_range:=0.9 max_range:=130.0 noise:=0.008 min_angle:=-${M_PI} max_angle:=${M_PI} gpu:=false">
+  <xacro:macro name="VLP-16" params="*origin parent:=upper_base_link name:=velodyne topic:=/velodyne_points hz:=20 lasers:=16 samples:=440 collision_range:=0.3 min_range:=0.9 max_range:=130.0 noise:=0.008 min_angle:=-${M_PI} max_angle:=${M_PI} gpu:=false visualize_sensor:=false">
     <joint name="${name}_base_mount_joint" type="fixed">
       <xacro:insert_block name="origin" />
@@ -58,5 +58,10 @@
         <sensor type="gpu_ray" name="${name}-VLP16">
           <pose>0 0 0 0 0 0</pose>
-          <visualize>false</visualize>
+          <xacro:if value="${visualize_sensor}">
+            <visualize>true</visualize>
+          </xacro:if>
+          <xacro:unless value="${visualize_sensor}">
+            <visualize>false</visualize>
+          </xacro:unless>
           <update_rate>${hz}</update_rate>
           <ray>
@@ -98,5 +103,10 @@
         <sensor type="ray" name="${name}-VLP16">
           <pose>0 0 0 0 0 0</pose>
-          <visualize>false</visualize>
+          <xacro:if value="${visualize_sensor}">
+            <visualize>true</visualize>
+          </xacro:if>
+          <xacro:unless value="${visualize_sensor}">
+            <visualize>false</visualize>
+          </xacro:unless>
           <update_rate>${hz}</update_rate>
           <ray>
